Commit message: Imported upstream version '3.0.0' of 'upstream'

File: crane_plus_description/urdf/camera.urdf.xacro (robot description, xacro)
@@ -6,11 +6,19 @@
         <origin xyz="0 0 0" rpy="0 0 0" />
         <geometry>
-          <box size="0.05 0.05 0.05" />
+          <box size="0.03 0.08 0.05" />
         </geometry>
-        <material name="Black" />
+        <material name="black">
+          <color rgba="0.2 0.2 0.2 1.0"/>
+        </material>
       </visual>
+      <collision>
+        <origin xyz="0 0 0" rpy="0 0 0"/>
+        <geometry>
+          <box size="0.03 0.08 0.05" />
+        </geometry>
+      </collision>
     </link>
     <joint name="camera_joint" type="fixed">
-      <origin xyz="0.103 0.1025 0.46" rpy="0 0 0" />
+      <origin xyz="0.10626 0.10253 0.46" rpy="0 0 0" />
       <parent link="${parent}" />
       <child link="camera_link" />

File: crane_plus_description/urdf/camera_stand.urdf.xacro (robot description, xacro)
@@ -6,5 +6,5 @@
         <origin xyz="0 0 0" rpy="0 0 0" />
         <geometry>
-          <box size="0.02 0.02 0.285" />
+          <box size="0.02 0.285 0.02" />
         </geometry>
         <material name="grey">
@@ -12,7 +12,13 @@
         </material>
       </visual>
+      <collision>
+        <origin xyz="0 0 0" rpy="0 0 0"/>
+        <geometry>
+          <box size="0.02 0.285 0.02" />
+        </geometry>
+      </collision>
     </link>
     <joint name="camera_stand_joint1" type="fixed">
-      <origin xyz="-0.05 0.08 0.01" rpy="${radians(90)} 0 0" />
+      <origin xyz="-0.052 0.08 0.01" rpy="0 0 0" />
       <parent link="${parent}" />
       <child link="camera_stand_p1" />
@@ -28,8 +34,14 @@
         </material>
       </visual>
+      <collision>
+        <origin xyz="0 0 0" rpy="0 0 0"/>
+        <geometry>
+          <box size="0.02 0.02 0.44" />
+        </geometry>
+      </collision>
     </link>
     <joint name="camera_stand_joint2" type="fixed">
-      <origin xyz="-0.05 0.1025 0.24" rpy="0 0 0" />
-      <parent link="${parent}" />
+      <origin xyz="0 0.02253 0.23" rpy="0 0 0" />
+      <parent link="camera_stand_p1" />
       <child link="camera_stand_p2" />
     </joint>
@@ -38,5 +50,5 @@
         <origin xyz="0 0 0" rpy="0 0 0" />
         <geometry>
-          <box size="0.02 0.02 0.13" />
+          <box size="0.13 0.02 0.02" />
         </geometry>
         <material name="grey">
@@ -44,8 +56,14 @@
         </material>
       </visual>
+      <collision>
+        <origin xyz="0 0 0" rpy="0 0 0"/>
+        <geometry>
+          <box size="0.129 0.02 0.02" />
+        </geometry>
+      </collision>
     </link>
     <joint name="camera_stand_joint3" type="fixed">
-      <origin xyz="0.02 0.1025 0.45" rpy="0 ${radians(90)} 0" />
-      <parent link="${parent}" />
+      <origin xyz="0.075 0 0.21" rpy="0 0 0" />
+      <parent link="camera_stand_p2" />
       <child link="camera_stand_p3" />
     </joint>
@@ -54,5 +72,5 @@
         <origin xyz="0 0 0" rpy="0 0 0" />
         <geometry>
-          <box size="0.02 0.02 0.05" />
+          <box size="0.055 0.02 0.02" />
         </geometry>
         <material name="grey">
@@ -60,8 +78,14 @@
         </material>
       </visual>
+      <collision>
+        <origin xyz="0 0 0" rpy="0 0 0"/>
+        <geometry>
+          <box size="0.054 0.019 0.02" />
+        </geometry>
+      </collision>
     </link>
     <joint name="camera_stand_joint4" type="fixed">
-      <origin xyz="-0.015 -0.0525 0.01" rpy="0 ${radians(90)} 0" />
-      <parent link="${parent}" />
+      <origin xyz="0.0375 -0.1325 0" rpy="0 0 0" />
+      <parent link="camera_stand_p1" />
       <child link="camera_stand_p4" />
     </joint>
@@ -70,5 +94,5 @@
         <origin xyz="0 0 0" rpy="0 0 0" />
         <geometry>
-          <box size="0.02 0.02 0.05" />
+          <box size="0.055 0.02 0.02" />
         </geometry>
         <material name="grey">
@@ -76,8 +100,14 @@
         </material>
       </visual>
+      <collision>
+        <origin xyz="0 0 0" rpy="0 0 0"/>
+        <geometry>
+          <box size="0.054 0.02 0.02" />
+        </geometry>
+      </collision>
     </link>
     <joint name="camera_stand_joint5" type="fixed">
-      <origin xyz="-0.015 0.2125 0.01" rpy="0 ${radians(90)} 0" />
-      <parent link="${parent}" />
+      <origin xyz="0.0375 0.1325 0" rpy="0 0 0" />
+      <parent link="camera_stand_p1" />
       <child link="camera_stand_p5" />
     </joint>

File: crane_plus_description/urdf/crane_plus.gazebo.xacro (robot description, xacro)
@@ -24,20 +24,12 @@
             name_link_4
             name_link_hand
-            use_ignition
+            use_camera
             config_package
             config_file_path
             ">
     <gazebo>
-      <xacro:if value="${use_ignition}">
-        <plugin filename="libign_ros2_control-system.so" name="ign_ros2_control::IgnitionROS2ControlPlugin">
-          <parameters>$(find ${config_package})/${config_file_path}</parameters>
-        </plugin>
-      </xacro:if>
-      <xacro:unless value="${use_ignition}">
-        <plugin filename="libgazebo_ros2_control.so" name="gazebo_ros2_control">
-          <robot_sim_type>gazebo_ros2_control/GazeboSystem</robot_sim_type>
-          <parameters>$(find ${config_package})/${config_file_path}</parameters>
-        </plugin>
-      </xacro:unless>
+      <plugin filename="libgz_ros2_control-system.so" name="gz_ros2_control::GazeboSimROS2ControlPlugin">
+      <parameters>$(find ${config_package})/${config_file_path}</parameters>
+      </plugin>
     </gazebo>
     <gazebo reference="${name_link_base}">
@@ -71,4 +63,52 @@
       <xacro:material_gazebo_white/>
     </gazebo>
+    <xacro:if value="$(arg use_camera)">
+      <gazebo>
+          <plugin filename="gz-sim-sensors-system" name="gz::sim::systems::Sensors">
+            <render_engine>ogre2</render_engine>
+          </plugin>
+      </gazebo>
+      <gazebo reference="camera_color_optical_frame">
+        <sensor name="camera" type="camera">
+          <pose relative_to="camera_color_optical_frame">0 0 0 ${radians(90)} ${radians(-90)} 0</pose>
+          <update_rate>10</update_rate>
+          <always_on>true</always_on>
+          <topic>image_raw</topic>
+          <gz_frame_id>camera_color_optical_frame</gz_frame_id>
+          <camera name="camera">
+            <xacro:property name="camera_width" value="640"/>
+            <xacro:property name="camera_height" value="480"/>
+            <xacro:property name="camera_hfov" value="${radians(70)}"/>
+            <xacro:property name="camera_focal_length" value="${camera_width / (2 * tan(camera_hfov / 2))}"/>
+            <horizontal_fov>${camera_hfov}</horizontal_fov>
+            <image>
+              <width>${camera_width}</width>
+              <height>${camera_height}</height>
+            </image>
+            <clip>
+              <near>0.1</near>
+              <far>10.0</far>
+            </clip>
+            <lens>
+              <intrinsics>
+                <fx>${camera_focal_length}</fx>
+                <fy>${camera_focal_length}</fy>
+                <cx>${(camera_width + 1) / 2}</cx>
+                <cy>${(camera_height + 1) / 2}</cy>
+                <s>1.0</s>
+              </intrinsics>
+              <projection>
+                <p_fx>${camera_focal_length}</p_fx>
+                <p_fy>${camera_focal_length}</p_fy>
+                <p_cx>${(camera_width + 1) / 2}</p_cx>
+                <p_cy>${(camera_height + 1) / 2}</p_cy>
+                <tx>0</tx>
+                <ty>0</ty>
+              </projection>
+            </lens>
+          </camera>
+        </sensor>
+      </gazebo>
+    </xacro:if>
   </xacro:macro>
 </robot>

File: crane_plus_description/urdf/crane_plus.gazebo_ros2_control.xacro (robot description, xacro)
@@ -18,14 +18,8 @@
             joint_hand_lower_limit
             joint_hand_upper_limit
-            use_ignition
             ">
     <ros2_control name="${name}" type="system">
       <hardware>
-        <xacro:if value="${use_ignition}">
-          <plugin>ign_ros2_control/IgnitionSystem</plugin>
-        </xacro:if>
-        <xacro:unless value="${use_ignition}">
-          <plugin>gazebo_ros2_control/GazeboSystem</plugin>
-        </xacro:unless>
+        <plugin>gz_ros2_control/GazeboSimSystem</plugin>
       </hardware>
       <joint name="${name_joint_1}">

File: crane_plus_description/urdf/crane_plus.ros2_control.xacro (robot description, xacro)
@@ -24,15 +24,21 @@
             read_loads
             read_voltages
-            read_temperatures">
+            read_temperatures
+            use_mock_components">
     <ros2_control name="${name}" type="system">
       <hardware>
-        <plugin>crane_plus_hardware/CranePlusHardware</plugin>
-        <param name="port_name">${port_name}</param>
-        <param name="baudrate">${baudrate}</param>
-        <param name="timeout_seconds">${timeout_seconds}</param>
-        <param name="read_velocities">${read_velocities}</param>
-        <param name="read_loads">${read_loads}</param>
-        <param name="read_voltages">${read_voltages}</param>
-        <param name="read_temperatures">${read_temperatures}</param>
+        <xacro:if value="${use_mock_components}">
+          <plugin>mock_components/GenericSystem</plugin>
+        </xacro:if>
+        <xacro:unless value="${use_mock_components}">
+          <plugin>crane_plus_hardware/CranePlusHardware</plugin>
+          <param name="port_name">${port_name}</param>
+          <param name="baudrate">${baudrate}</param>
+          <param name="timeout_seconds">${timeout_seconds}</param>
+          <param name="read_velocities">${read_velocities}</param>
+          <param name="read_loads">${read_loads}</param>
+          <param name="read_voltages">${read_voltages}</param>
+          <param name="read_temperatures">${read_temperatures}</param>
+        </xacro:unless>
       </hardware>
       <joint name="${name_joint_1}">

File: crane_plus_description/urdf/crane_plus.urdf.xacro (robot description, xacro)
@@ -11,6 +11,6 @@
   <xacro:include filename="$(find crane_plus_description)/urdf/crane_plus.gazebo_ros2_control.xacro"/>
   <xacro:arg name="use_gazebo" default="false" />
-  <xacro:arg name="use_ignition" default="false" />
   <xacro:arg name="use_camera" default="false" />
+  <xacro:arg name="use_mock_components" default="false" />
   <xacro:arg name="port_name" default="/dev/ttyUSB0" />
   <xacro:arg name="baudrate" default="1000000" />
@@ -108,5 +108,6 @@
       read_loads="$(arg read_loads)"
       read_voltages="$(arg read_voltages)"
-      read_temperatures="$(arg read_temperatures)" />
+      read_temperatures="$(arg read_temperatures)"
+      use_mock_components="$(arg use_mock_components)" />
   </xacro:unless>
   <xacro:if value="$(arg use_gazebo)">
@@ -118,5 +119,5 @@
       name_link_4="${NAME_LINK_4}"
       name_link_hand="${NAME_LINK_HAND}"
-      use_ignition="$(arg use_ignition)"
+      use_camera="$(arg use_camera)"
       config_package="$(arg gz_control_config_package)"
       config_file_path="$(arg gz_control_config_file_path)" />
@@ -137,6 +138,5 @@
       joint_4_upper_limit="${JOINT_4_UPPER_LIMIT}"
       joint_hand_lower_limit="${JOINT_HAND_LOWER_LIMIT}"
-      joint_hand_upper_limit="${JOINT_HAND_UPPER_LIMIT}"
-      use_ignition="$(arg use_ignition)" />
+      joint_hand_upper_limit="${JOINT_HAND_UPPER_LIMIT}"/>
   </xacro:if>
 </robot>
